File: KiCad/Le Chiffre v2/LeChiffre.kicad_pcb (KiCad board)
At the start: 2 copper layers, 228.4 x 85 mm, 105 parts, among them J1 Conn_01x03_Female, J2 Conn_01x04_Female, SW1 SW_Push, SW10 SW_Push, SW11 SW_Push, SW12 SW_Push, SW13 SW_Push, SW14 SW_Push, SW15 SW_Push, SW16 SW_Push, SW17 SW_Push, SW18 SW_Push, SW19 SW_Push, SW2 SW_Push, SW20 SW_Push, SW21 SW_Push, SW22 SW_Push, SW23 SW_Push, SW24 SW_Push, SW25 SW_Push, SW26 SW_Push, SW27 SW_Push, SW28 SW_Push, SW29 SW_Push, SW3 SW_Push, SW30 SW_Push, SW31 SW_Push, SW32 SW_Push, SW33 SW_Push, SW34 SW_Push, SW35 SW_Push, SW36 Rotary_Encoder_Switch, SW37 SW_Push, SW4 SW_Push, SW5 SW_Push, SW6 SW_Push, SW7 SW_Push, SW8 SW_Push, SW9 SW_Push, U1 ATmega32U4-AU, Y1 Crystal_GND2

Commit message: First commit, removing vias and tracks and mcu, adding nice_nano/supermioni/promicro
Parts:
- removed C1, C2, C5, C7: .1u, Keebio-Parts:C_0603
- removed C3, C6: 22p, Keebio-Parts:C_0603
- removed C4: 1u, Keebio-Parts:C_0603
- removed C8: 4.7u, Keebio-Parts:C_0603
- removed D101, D102, D103, D104, D105, D106, D107, D108, D109, D110, D111: WS2812B, LED_SMD:LED_WS2812B_PLCC4_5.0x5.0mm_P3.2mm
- removed F1: Polyfuse_Small, Keebio-Parts:Fuse_0805
- removed J1: Conn_01x03_Female, Connector_PinSocket_2.54mm:PinSocket_1x03_P2.54mm_Vertical
- removed J2: Conn_01x04_Female, Connector_PinSocket_2.54mm:PinSocket_1x04_P2.54mm_Vertical
- removed R1, R2: 5.1k, Keebio-Parts:R_0805
- removed R3, R4: 22, Keebio-Parts:R_0805
- removed R5, R6: 10k, Keebio-Parts:R_0805
- removed R7, R8: 4.7k, Keebio-Parts:R_0805
- removed SW1: SW_Push, Keebio-Parts:SW_SPST_TL3342
- removed SW37: SW_Push, Keebio-Parts:MX-Alps-Choc-1U-NoLED
- removed USB1: HRO-TYPE-C-31-M-12, Type-C:HRO-TYPE-C-31-M-12-HandSoldering
- removed Y1: Crystal_GND2, Keebio-Parts:Crystal_SMD_3225-4pin_3.2x2.5mm
- U1: value ATmega32U4-AU -> SuperMini nRF52840 x nice_nano; footprint Keebio-Parts:ATMEGA32U4-AU -> pro_micro:supermini_x_nice_nano; moved to F.Cu
- moved U1 61.7 mm to (138.1, 46.0)
- moved SW36 33.8 mm to (135.9, 101.2)
- moved D35 33.8 mm to (148.7, 97.8)
Connections:
- U1 pad 1: Net-(U1-Pad1) -> unconnected-(U1-P0.06-Pad1)
- U1 pad 10: col3 -> row3
- U1 pad 11: row0 -> col0
- U1 pad 12: Net-(U1-Pad12) -> col1
- U1 pad 13: Net-(R5-Pad2) -> unconnected-(U1-BAT+-Pad13)
- U1 pad 14: VCC -> GND
- U1 pad 15: GND -> unconnected-(U1-RST-Pad15)
- U1 pad 16: Net-(C6-Pad1) -> unconnected-(U1-3V3-Pad16)
- U1 pad 17: Net-(C3-Pad1) -> col2
- U1 pad 18: SCK -> col3
- U1 pad 19: SDA -> col4
- U1 pad 2: VCC -> unconnected-(U1-P0.08-Pad2)
- U1 pad 20: col8 -> col5
- U1 pad 21: EncB -> col6
- U1 pad 22: EncA -> col7
- U1 pad 23: GND -> col8
- U1 pad 24: VCC -> col9
- U1 pad 25: row1 -> unconnected-(U1-P1.01-LF-Pad25)
- U1 pad 26: Net-(U1-Pad26) -> unconnected-(U1-P1.02-LF-Pad26)
- U1 pad 27: col6 -> unconnected-(U1-P1.07-LF-Pad27)
- U1 pad 28: col5 -> GND
- U1 pad 29: Net-(U1-Pad29) -> unconnected-(U1-BAT+-Pad29)
- U1 pad 3: /D- -> GND
- U1 pad 4: /D+ -> GND
- U1 pad 5: GND -> EncA
- U1 pad 6: UCAP -> EncB
- U1 pad 7: VCC -> row0
- U1 pad 8: col2 -> row1
- U1 pad 9: col4 -> row2
Routing:
- net VCC: track 698.2 -> 0.00 mm, vias 13 -> 0
- net row0: track 263.9 -> 0.00 mm, vias 3 -> 0
- net row2: track 252.5 -> 0.00 mm, vias 2 -> 0
- net row1: track 234.4 -> 0.00 mm
- net row3: track 218.9 -> 0.00 mm, vias 3 -> 0
- net col8: track 186.3 -> 0.00 mm, vias 2 -> 0
- net col0: track 185.9 -> 0.00 mm, vias 1 -> 0
- net col9: track 174.6 -> 0.00 mm, vias 1 -> 0
- net col7: track 155.4 -> 0.00 mm
- net col1: track 152.9 -> 0.00 mm, vias 3 -> 0
- net col2: track 148.1 -> 0.00 mm, vias 2 -> 0
- net col5: track 105.8 -> 0.00 mm
- net col6: track 101.8 -> 0.00 mm
- net col3: track 99.1 -> 0.00 mm
- net col4: track 95.2 -> 0.00 mm, vias 1 -> 0
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- removed copper zone on B.Cu, net GND
- removed copper zone on F.Cu, net GND
Other:
- board size 228.4 x 85 mm -> 228.4 x 84.9 mm
- net class Default removed
- net class power removed
- board text removed: "PF0"
